File: pcbs/adapters/adapters.kicad_pcb (KiCad board)
At the start: 2 copper layers, 99 x 95 mm, 13 parts, among them J1 USB_B, J10 Conn_01x05_Pin, J11 Conn_01x06_Socket, J12 Conn_01x06_Socket, J13 Conn_01x04_Pin, J2 USB_B, J3 DA15_Pins_MountingHoles, J4 Conn_01x06_Pin, J5 Conn_01x06_Pin, J6 Conn_01x05_Pin, J7 Conn_01x05_Pin, J8 Conn_01x06_Pin, J9 Conn_01x06_Pin

Commit message: first rough version of top board
Parts:
- removed J6, J7: Conn_01x05_Pin, Connector_PinHeader_2.54mm:PinHeader_1x05_P2.54mm_Vertical
- removed J8: Conn_01x06_Pin, Connector_JST:JST_XA_S06B-XASK-1_1x06_P2.50mm_Horizontal
- removed J9: Conn_01x06_Pin, Connector_PinHeader_2.54mm:PinHeader_1x06_P2.54mm_Vertical
- added F5: f5, Connector_Wire:SolderWire-1.5sqmm_1x01_D1.7mm_OD3mm, F.Cu at (103.0, 74.3)
- added FID4: Fiducial, Fiducial:Fiducial_0.5mm_Mask2mm, F.Cu at (196.5, 143.2)
- added FID5: Fiducial, Fiducial:Fiducial_0.5mm_Mask2mm, F.Cu at (90.0, 134.2)
- added FID6: Fiducial, Fiducial:Fiducial_0.5mm_Mask2mm, F.Cu at (118.5, 52.7)
- added H1: MountingHole, MountingHole:MountingHole_3.2mm_M3_Pad_TopBottom, F.Cu at (89.0, 53.7)
- added H2: MountingHole, MountingHole:MountingHole_3.2mm_M3_Pad_TopBottom, F.Cu at (89.5, 144.7)
- added H3: MountingHole, MountingHole:MountingHole_3.2mm_M3_Pad_TopBottom, F.Cu at (211.0, 144.7)
- added H4: MountingHole, MountingHole:MountingHole_3.2mm_M3_Pad_TopBottom, F.Cu at (211.0, 53.7)
- added J14: Conn_01x04_Pin, Connector_PinHeader_2.54mm:PinHeader_1x04_P2.54mm_Vertical, F.Cu at (128.2, 79.0)
- added J15: Conn_01x06_Pin, Connector_PinHeader_2.54mm:PinHeader_1x06_P2.54mm_Vertical, F.Cu at (209.0, 96.0)
- added J16: f4, Connector_Wire:SolderWire-1.5sqmm_1x01_D1.7mm_OD3mm, F.Cu at (108.1, 59.5)
- added J17: f6, Connector_Wire:SolderWire-1.5sqmm_1x01_D1.7mm_OD3mm, F.Cu at (108.1, 82.3)
- added J18: f6, Connector_Wire:SolderWire-1.5sqmm_1x01_D1.7mm_OD3mm, F.Cu at (103.0, 82.3)
- added J19: f5, Connector_Wire:SolderWire-1.5sqmm_1x01_D1.7mm_OD3mm, F.Cu at (108.1, 74.3)
- added J1_probe1: USB_B, Connector_USB:USB_B_Lumberg_2411_02_Horizontal, F.Cu at (106.2, 128.8)
- added J21_240V_IN1: Screw_Terminal_01x02, TerminalBlock_Phoenix:TerminalBlock_Phoenix_MKDS-1-2-3.81_1x02_P3.81mm_Horizontal, F.Cu at (92.0, 76.5)
- added J22_240V_OUT1: Screw_Terminal_01x02, TerminalBlock_Phoenix:TerminalBlock_Phoenix_MKDS-1-2-3.81_1x02_P3.81mm_Horizontal, F.Cu at (92.5, 61.2)
- added J23: f2, Connector_Wire:SolderWire-1.5sqmm_1x01_D1.7mm_OD3mm, F.Cu at (108.1, 101.4)
- added J24: f2, Connector_Wire:SolderWire-1.5sqmm_1x01_D1.7mm_OD3mm, F.Cu at (103.0, 101.4)
- added J25: f1, Connector_Wire:SolderWire-1.5sqmm_1x01_D1.7mm_OD3mm, F.Cu at (108.2, 109.0)
- added J26: f1, Connector_Wire:SolderWire-1.5sqmm_1x01_D1.7mm_OD3mm, F.Cu at (103.1, 109.0)
- added J27_24V_in1: Screw_Terminal_01x02, TerminalBlock_Phoenix:TerminalBlock_Phoenix_MKDS-1-2-3.81_1x02_P3.81mm_Horizontal, F.Cu at (92.5, 103.5)
- added J2_Spindle1: USB_B, Connector_USB:USB_B_Lumberg_2411_02_Horizontal, F.Cu at (130.7, 69.1)
- added J4_X2: Conn_01x06_Pin, Connector_JST:JST_VH_S6P-VH_1x06_P3.96mm_Horizontal, F.Cu at (153.7, 130.2)
- added J5_X1: Conn_01x06_Pin, Connector_JST:JST_VH_S6P-VH_1x06_P3.96mm_Horizontal, F.Cu at (125.7, 130.2)
- added J8_Z1: Conn_01x06_Pin, Connector_JST:JST_XA_S06B-XASK-1_1x06_P2.50mm_Horizontal, F.Cu at (154.5, 68.2)
- added J9_End_Stops1: Conn_01x06_Pin, Connector_JST:JST_XA_S06B-XASK-1_1x06_P2.50mm_Horizontal, F.Cu at (198.5, 83.5)
- J1, J2: value USB_B -> Screw_Terminal_01x06; footprint Connector_USB:USB_B_Lumberg_2411_02_Horizontal -> TerminalBlock_Phoenix:TerminalBlock_Phoenix_MKDS-1-6-3.81_1x06_P3.81mm_Horizontal
- J10: value Conn_01x05_Pin -> f3; footprint Connector_PinHeader_2.54mm:PinHeader_1x05_P2.54mm_Vertical -> Connector_Wire:SolderWire-1.5sqmm_1x01_D1.7mm_OD3mm
- J11: value Conn_01x06_Socket -> f3; footprint Connector_Phoenix_MSTB:PhoenixContact_MSTBA_2,5_6-G-5,08_1x06_P5.08mm_Horizontal -> Connector_Wire:SolderWire-1.5sqmm_1x01_D1.7mm_OD3mm
- J12: value Conn_01x06_Socket -> f4; footprint Connector_Phoenix_MSTB:PhoenixContact_MSTBA_2,5_6-G-5,08_1x06_P5.08mm_Horizontal -> Connector_Wire:SolderWire-1.5sqmm_1x01_D1.7mm_OD3mm
- J3: value DA15_Pins_MountingHoles -> DA15_Bottom; footprint Connector_Dsub:DSUB-15-HD_Pins_Horizontal_P2.29x1.90mm_EdgePinOffset3.03mm_Housed_MountingHolesOffset4.94mm -> Connector_Dsub:DSUB-15-HD_Socket_Horizontal_P2.29x1.90mm_EdgePinOffset3.03mm_Housed_MountingHolesOffset4.94mm
- J4: value Conn_01x06_Pin -> Screw_Terminal_01x06; footprint Connector_JST:JST_VH_S6P-VH_1x06_P3.96mm_Horizontal -> TerminalBlock_Phoenix:TerminalBlock_Phoenix_MKDS-1-6-3.81_1x06_P3.81mm_Horizontal
- J5: value Conn_01x06_Pin -> Conn_02x08_Counter_Clockwise; footprint Connector_JST:JST_VH_S6P-VH_1x06_P3.96mm_Horizontal -> Connector_PinHeader_2.54mm:PinHeader_2x08_P2.54mm_Vertical
- moved J5 93.9 mm to (191.0, 112.9), turned to 0 degrees
- moved J3 77.5 mm to (207.1, 118.2), turned to 90 degrees
- moved J4 73.1 mm to (170.3, 55.7), turned to 180 degrees
- moved J11 56.8 mm to (103.0, 67.0), turned to 0 degrees
- moved J13 39.0 mm to (108.5, 118.2), turned to -90 degrees
- moved J10 38.4 mm to (108.1, 67.0), turned to 0 degrees
- moved J2 32.4 mm to (173.1, 120.7), turned to 180 degrees
- moved J12 23.5 mm to (103.0, 59.5), turned to 0 degrees
- moved J1 14.9 mm to (145.1, 120.7), turned to 180 degrees
Connections:
- J1 pad 1: Net-(J1-VBUS) -> Net-(J1-Pin_1)
- J1 pad 2: Net-(J1-D-) -> Net-(J1-Pin_2)
- J1 pad 3: Net-(J1-D+) -> Net-(J1-Pin_3)
- J1 pad 4: GNDREF -> Net-(J1-Pin_4)
- J11 pad 1: Net-(J11-Pin_1) -> Net-(J10-Pin_1)
- J13 pad 1: GNDREF -> GND
- J13 pad 2: Net-(J1-D-) -> Net-(J13-Pin_2)
- J13 pad 3: Net-(J1-D+) -> Net-(J13-Pin_3)
- J13 pad 4: Net-(J1-VBUS) -> Net-(J13-Pin_4)
- J2 pad 4: GNDREF -> Net-(J2-Pin_4)
- J3 pad 1: Net-(J10-Pin_5) -> Net-(J5-Pin_8)
- J3 pad 10: Net-(J10-Pin_2) -> Net-(J3-P10)
- J3 pad 2: Net-(J10-Pin_3) -> Net-(J5-Pin_10)
- J3 pad 3: Net-(J10-Pin_1) -> Net-(J5-Pin_12)
- J3 pad 4: Net-(J7-Pin_4) -> Net-(J5-Pin_14)
- J3 pad 5: Net-(J7-Pin_2) -> Net-(J5-Pin_16)
- J3 pad 6: Net-(J6-Pin_5) -> Net-(J5-Pin_7)
- J3 pad 7: Net-(J6-Pin_3) -> Net-(J5-Pin_9)
- J3 pad 8: GNDREF -> Net-(J5-Pin_11)
- J3 pad 9: Net-(J10-Pin_4) -> Net-(J3-P9)
- J3 pad SH: unconnected-(J3-PAD-PadSH) -> GND
- J4 pad 1: Net-(J12-Pin_1) -> Net-(J4-Pin_1)
- J4 pad 2: Net-(J12-Pin_2) -> Net-(J4-Pin_2)
- J4 pad 3: Net-(J12-Pin_3) -> Net-(J4-Pin_3)
- J4 pad 4: Net-(J12-Pin_4) -> Net-(J4-Pin_4)
- J4 pad 5: Net-(J12-Pin_5) -> Net-(J4-Pin_5)
- J4 pad 6: Net-(J12-Pin_6) -> Net-(J4-Pin_6)
- J5 pad 1: Net-(J11-Pin_1) -> Net-(J3-P14)
- J5 pad 2: Net-(J11-Pin_2) -> Net-(J3-P13)
- J5 pad 3: Net-(J11-Pin_3) -> Net-(J3-P15)
- J5 pad 4: Net-(J11-Pin_4) -> Net-(J3-P12)
- J5 pad 5: Net-(J11-Pin_5) -> unconnected-(J5-Pin_5-Pad5)
- J5 pad 6: Net-(J11-Pin_6) -> Net-(J3-P111)
Routing:
- net GND: track 0.00 -> 300.6 mm
- net (no net): track 53.0 -> 0.00 mm
- net Net-(J3-P15): track 0.00 -> 41.5 mm
- net Net-(J3-P14): track 0.00 -> 33.1 mm
- net Net-(J3-P13): track 0.00 -> 26.7 mm
- net Net-(J3-P12): track 0.00 -> 23.0 mm
- net Net-(J3-P10): track 0.00 -> 19.9 mm
- net Net-(J3-P9): track 0.00 -> 19.8 mm
- net Net-(J5-Pin_11): track 0.00 -> 19.7 mm
- net Net-(J3-P111): track 0.00 -> 19.6 mm
- net Net-(J5-Pin_9): track 0.00 -> 19.6 mm
- net Net-(J5-Pin_7): track 0.00 -> 19.5 mm
- net Net-(F5-Pin_1): track 0.00 -> 17.1 mm
- net Net-(J17-Pin_1): track 0.00 -> 17.0 mm
- net Net-(J10-Pin_1): track 0.00 -> 16.5 mm
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Other:
- board size 99 x 95 mm -> 130 x 99.5 mm
- rule pad_to_mask_clearance: 0 -> 0.1
