File: pcbs/adapters/adapters.kicad_sch (KiCad schematic)
At the start: 14 parts, among them J1 USB_B, J10 Conn_01x05_Pin, J11 Conn_01x06_Socket, J12 Conn_01x06_Socket, J13 Conn_01x04_Pin, J14 Conn_01x04_Pin, J2 USB_B, J3 DA15_Pins_MountingHoles, J4 Conn_01x06_Pin, J5 Conn_01x06_Pin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

Commit message: PCB draft tweaks + ignores
Parts:
- removed J11, J12: Conn_01x06_Socket, Connector_Phoenix_MSTB:PhoenixContact_MSTBA_2,5_6-G-5,08_1x06_P5.08mm_Horizontal, symbol Connector:Conn_01x06_Socket
- removed J9: Conn_01x06_Pin, Connector_PinHeader_2.54mm:PinHeader_1x06_P2.54mm_Vertical, symbol Connector:Conn_01x06_Pin
- added J1, J2, J4: Screw_Terminal_01x06, TerminalBlock_Phoenix:TerminalBlock_Phoenix_MKDS-1-6-3.81_1x06_P3.81mm_Horizontal, symbol Connector:Screw_Terminal_01x06
- added J15: Conn_01x06_Pin, Connector_PinHeader_2.54mm:PinHeader_1x06_P2.54mm_Vertical, symbol Connector:Conn_01x06_Pin
- added J9_ES1: Conn_01x06_Pin, Connector_JST:JST_XA_S06B-XASK-1_1x06_P2.50mm_Horizontal, symbol Connector:Conn_01x06_Pin
- J3: value DA15_Pins_MountingHoles -> DA15_Bottom
- renumbered J1 to J1_probe1, J2 to J2_Spindle1, J4 to J4_X2, J5 to J5_X1, J8 to J8_Z1
Connections:
- net at J5_X1.1 (Pin_1): now also J1.1 (Pin_1)
- net at J5_X1.2 (Pin_2): now also J1.2 (Pin_2)
- net at J5_X1.3 (Pin_3): now also J1.3 (Pin_3)
- net at J5_X1.4 (Pin_4): now also J1.4 (Pin_4)
- net at J5_X1.5 (Pin_5): now also J1.5 (Pin_5)
- net at J5_X1.6 (Pin_6): now also J1.6 (Pin_6)
- net at J4_X2.1 (Pin_1): now also J2.1 (Pin_1)
- net at J4_X2.2 (Pin_2): now also J2.2 (Pin_2)
- net at J4_X2.3 (Pin_3): now also J2.3 (Pin_3)
- net at J4_X2.4 (Pin_4): now also J2.4 (Pin_4)
- net at J4_X2.5 (Pin_5): now also J2.5 (Pin_5)
- net at J4_X2.6 (Pin_6): now also J2.6 (Pin_6)
- net at J8_Z1.1 (Pin_1): now also J4.1 (Pin_1)
- net at J8_Z1.2 (Pin_2): now also J4.2 (Pin_2)
- net at J8_Z1.3 (Pin_3): now also J4.3 (Pin_3)
- net at J8_Z1.4 (Pin_4): now also J4.4 (Pin_4)
- net at J8_Z1.5 (Pin_5): now also J4.5 (Pin_5)
- net at J8_Z1.6 (Pin_6): now also J4.6 (Pin_6)
- new net: J15.6 (Pin_6), J9_ES1.1 (Pin_1)
- new net: J15.5 (Pin_5), J9_ES1.2 (Pin_2)
- new net: J15.4 (Pin_4), J9_ES1.3 (Pin_3)
- new net: J15.3 (Pin_3), J9_ES1.4 (Pin_4)
- new net: J15.2 (Pin_2), J9_ES1.5 (Pin_5)
- new net: J15.1 (Pin_1), J9_ES1.6 (Pin_6)
Other:
- moved on the sheet: J10, J3, J4_X2, J5_X1, J6, J7, J8_Z1

Commit message: first rough version of top board
Parts:
- removed J10, J6, J7: Conn_01x05_Pin, Connector_PinHeader_2.54mm:PinHeader_1x05_P2.54mm_Vertical, symbol Connector:Conn_01x05_Pin
- added F5, J19: f5, Connector_Wire:SolderWire-1.5sqmm_1x01_D1.7mm_OD3mm, symbol Connector:Conn_01x01_Socket
- added FID4, FID5, FID6: Fiducial, Fiducial:Fiducial_0.5mm_Mask2mm, symbol Mechanical:Fiducial
- added H1, H2, H3, H4: MountingHole, MountingHole:MountingHole_3.2mm_M3_Pad_TopBottom, symbol Mechanical:MountingHole
- added J10, J11: f3, Connector_Wire:SolderWire-1.5sqmm_1x01_D1.7mm_OD3mm, symbol Connector:Conn_01x01_Socket
- added J12, J16: f4, Connector_Wire:SolderWire-1.5sqmm_1x01_D1.7mm_OD3mm, symbol Connector:Conn_01x01_Socket
- added J17, J18: f6, Connector_Wire:SolderWire-1.5sqmm_1x01_D1.7mm_OD3mm, symbol Connector:Conn_01x01_Socket
- added J21_240V_IN1, J22_240V_OUT1, J27_24V_in1: Screw_Terminal_01x02, TerminalBlock_Phoenix:TerminalBlock_Phoenix_MKDS-1-2-3.81_1x02_P3.81mm_Horizontal, symbol Connector:Screw_Terminal_01x02
- added J23, J24: f2, Connector_Wire:SolderWire-1.5sqmm_1x01_D1.7mm_OD3mm, symbol Connector:Conn_01x01_Socket
- added J25, J26: f1, Connector_Wire:SolderWire-1.5sqmm_1x01_D1.7mm_OD3mm, symbol Connector:Conn_01x01_Socket
- added J5: Conn_02x08_Counter_Clockwise, Connector_PinHeader_2.54mm:PinHeader_2x08_P2.54mm_Vertical, symbol Connector_Generic:Conn_02x08_Counter_Clockwise
- J14: footprint (none) -> Connector_PinHeader_2.54mm:PinHeader_1x04_P2.54mm_Vertical
- J3: footprint Connector_Dsub:DSUB-15-HD_Pins_Horizontal_P2.29x1.90mm_EdgePinOffset3.03mm_Housed_MountingHolesOffset4.94mm -> Connector_Dsub:DSUB-15-HD_Socket_Horizontal_P2.29x1.90mm_EdgePinOffset3.03mm_Housed_MountingHolesOffset4.94mm
- renumbered J9_ES1 to J9_End_Stops1
Connections:
- net at J2_Spindle1.1 (VBUS): now also J14.2 (Pin_2); no longer J14.4 (Pin_4)
- net at J2_Spindle1.2 (D-): now also J14.3 (Pin_3); no longer J14.2 (Pin_2)
- net at J2_Spindle1.3 (D+): now also J14.4 (Pin_4); no longer J14.3 (Pin_3)
- net at J13.2 (Pin_2): now also J1_probe1.1 (VBUS); no longer J1_probe1.2 (D-)
- net at J13.3 (Pin_3): now also J1_probe1.2 (D-); no longer J1_probe1.3 (D+)
- net at J13.4 (Pin_4): now also J1_probe1.3 (D+); no longer J1_probe1.1 (VBUS)
- net at J3.1: now also J5.8 (Pin_8)
- net at J3.10 (P10): now also J5.15 (Pin_15)
- net at J3.11 (P111): now also J5.6 (Pin_6)
- net at J3.12 (P12): now also J5.4 (Pin_4)
- net at J3.13 (P13): now also J5.2 (Pin_2)
- net at J3.14 (P14): now also J5.1 (Pin_1)
- net at J3.15 (P15): now also J5.3 (Pin_3)
- net at J3.2: now also J5.10 (Pin_10)
- net at J3.3: now also J5.12 (Pin_12)
- net at J3.4: now also J5.14 (Pin_14)
- net at J3.5: now also J5.16 (Pin_16)
- net at J3.6: now also J5.7 (Pin_7)
- net at J3.7: now also J5.9 (Pin_9)
- net at J3.9 (P9): now also J5.13 (Pin_13)
- net GND: now reaches J3.SH (PAD)
- net GND: now also J13.1 (Pin_1), J14.1 (Pin_1), J1_probe1.4 (GND), J1_probe1.SH (Shield), J2_Spindle1.4 (GND), J2_Spindle1.SH (Shield)
- net at J2.1 (Pin_1): now also J4_X2.6 (Pin_6); no longer J4_X2.1 (Pin_1)
- net at J2.2 (Pin_2): now also J4_X2.5 (Pin_5); no longer J4_X2.2 (Pin_2)
- net at J2.3 (Pin_3): now also J4_X2.4 (Pin_4); no longer J4_X2.3 (Pin_3)
- net at J2.4 (Pin_4): now also J4_X2.3 (Pin_3); no longer J4_X2.4 (Pin_4)
- net at J2.5 (Pin_5): now also J4_X2.2 (Pin_2); no longer J4_X2.5 (Pin_5)
- net at J2.6 (Pin_6): now also J4_X2.1 (Pin_1); no longer J4_X2.6 (Pin_6)
- net at J1.1 (Pin_1): now also J5_X1.6 (Pin_6); no longer J5_X1.1 (Pin_1)
- net at J1.2 (Pin_2): now also J5_X1.5 (Pin_5); no longer J5_X1.2 (Pin_2)
- net at J1.3 (Pin_3): now also J5_X1.4 (Pin_4); no longer J5_X1.3 (Pin_3)
- net at J1.4 (Pin_4): now also J5_X1.3 (Pin_3); no longer J5_X1.4 (Pin_4)
- net at J1.5 (Pin_5): now also J5_X1.2 (Pin_2); no longer J5_X1.5 (Pin_5)
- net at J1.6 (Pin_6): now also J5_X1.1 (Pin_1); no longer J5_X1.6 (Pin_6)
- net at J8_Z1.1 (Pin_1): now also J4.6 (Pin_6); no longer J4.1 (Pin_1)
- net at J8_Z1.2 (Pin_2): now also J4.5 (Pin_5); no longer J4.2 (Pin_2)
- net at J8_Z1.3 (Pin_3): now also J4.4 (Pin_4); no longer J4.3 (Pin_3)
- net at J8_Z1.4 (Pin_4): now also J4.3 (Pin_3); no longer J4.4 (Pin_4)
- net at J8_Z1.5 (Pin_5): now also J4.2 (Pin_2); no longer J4.5 (Pin_5)
- net at J8_Z1.6 (Pin_6): now also J4.1 (Pin_1); no longer J4.6 (Pin_6)
- removed net GNDREF: J13.1 (Pin_1), J14.1 (Pin_1), J1_probe1.4 (GND), J1_probe1.SH (Shield), J2_Spindle1.4 (GND), J2_Spindle1.SH (Shield), J3.8
- new net: J25.1 (Pin_1), J26.1 (Pin_1), J27_24V_in1.2 (Pin_2)
- new net: F5.1 (Pin_1), J19.1 (Pin_1), J21_240V_IN1.1 (Pin_1)
- new net: J3.8, J5.11 (Pin_11)
- new net: J17.1 (Pin_1), J18.1 (Pin_1), J21_240V_IN1.2 (Pin_2)
- new net: J23.1 (Pin_1), J24.1 (Pin_1), J27_24V_in1.1 (Pin_1)
- new net: J12.1 (Pin_1), J16.1 (Pin_1), J22_240V_OUT1.1 (Pin_1)
- new net: J10.1 (Pin_1), J11.1 (Pin_1), J22_240V_OUT1.2 (Pin_2)
Other:
- company: (none) -> Kakwalab
- title: (none) -> Yeti Adapter Board
- moved on the sheet: J1, J13, J1_probe1, J2, J2_Spindle1, J3, J4, J4_X2, J5_X1
