File: pcbs/breakout_top_dsub25/adapters.kicad_sch (KiCad schematic)
At the start: 37 parts, among them J1 Screw_Terminal_01x06, J10 f3, J11 f3, J12 f4, J13 Conn_01x04_Pin, J14 Conn_01x04_Pin, J15 Conn_01x06_Pin, J16 f4, J17 f6, J18 f6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

Commit message: relabel dsub 25 pins which were rewired/renumbered for 24V routing + add spacing for power supply stuff.
Parts:
- J21_240V_IN1, J22_240V_OUT1, J27_24V_in1: footprint TerminalBlock_Phoenix:TerminalBlock_Phoenix_MKDS-1-2-3.81_1x02_P3.81mm_Horizontal -> TerminalBlock_Phoenix:TerminalBlock_Phoenix_MKDS-1,5-2_1x02_P5.00mm_Horizontal
- J8_Z1, J9_End_Stops1: footprint Connector_JST:JST_XA_S06B-XASK-1_1x06_P2.50mm_Horizontal -> Connector_JST:JST_XA_S06B-XASK-1N-BN_1x06_P2.50mm_Horizontal
Changed lines of the file:
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@@
 		(title "Yeti Adapter Board")
 		(date "2026-04-29")
-		(rev "0")
+		(rev "2")
 		(company "Kakwalab")
 	)
@@
 			)
 		)
-		(property "Footprint" "TerminalBlock_Phoenix:TerminalBlock_Phoenix_MKDS-1-2-3.81_1x02_P3.81mm_Horizontal"
+		(property "Footprint" "TerminalBlock_Phoenix:TerminalBlock_Phoenix_MKDS-1,5-2_1x02_P5.00mm_Horizontal"
 			(at 130.81 30.48 0)
 			(hide yes)
@@
 			)
 		)
-		(property "Footprint" "Connector_JST:JST_XA_S06B-XASK-1_1x06_P2.50mm_Horizontal"
+		(property "Footprint" "Connector_JST:JST_XA_S06B-XASK-1N-BN_1x06_P2.50mm_Horizontal"
 			(at 130.81 119.38 0)
 			(hide yes)
@@
 			)
 		)
-		(property "Footprint" "TerminalBlock_Phoenix:TerminalBlock_Phoenix_MKDS-1-2-3.81_1x02_P3.81mm_Horizontal"
+		(property "Footprint" "TerminalBlock_Phoenix:TerminalBlock_Phoenix_MKDS-1,5-2_1x02_P5.00mm_Horizontal"
 			(at 128.27 52.07 0)
 			(hide yes)
@@
 			)
 		)
-		(property "Footprint" "Connector_JST:JST_XA_S06B-XASK-1_1x06_P2.50mm_Horizontal"
+		(property "Footprint" "Connector_JST:JST_XA_S06B-XASK-1N-BN_1x06_P2.50mm_Horizontal"
 			(at 54.61 72.39 0)
 			(hide yes)
@@
 			)
 		)
-		(property "Footprint" "TerminalBlock_Phoenix:TerminalBlock_Phoenix_MKDS-1-2-3.81_1x02_P3.81mm_Horizontal"
+		(property "Footprint" "TerminalBlock_Phoenix:TerminalBlock_Phoenix_MKDS-1,5-2_1x02_P5.00mm_Horizontal"
 			(at 129.54 76.2 0)
 			(hide yes)
